File: Hardware/Proiect_TSC_2025 v39.sch (EAGLE design)
At the start: 103 parts, among them IC1 BD5229G-TR, IC4 XC6220A331MR-G, J1 FH34SRJ-24S-0.5SH_99_, J2 SAMACSYS_PARTS_USB4110-GF-A, J3 QWIIC_RIGHT_ANGLE, J4 112A-TAAR-R03_ATTEND, Q1 20V/4.2A/52mΩ/1.4W, Q2 20V/4.2A/52mΩ/1.4W, Q3 SI1308EDL-T1-GE3, U1 W25Q512JVEIQ, U2 ESP32-C6-WROOM-1-N8, U3 DS3231SN#, U4 MAX17048G+T10

Commit message: Fixed issues
Connections:
- removed net N$4: EPD_C9.2, J1.21
- net PREVGH: now also EPD_C9.2, J1.21
Changed lines of the file:
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@@
 </segment>
 </net>
-<net name="N$4" class="2">
+<net name="PREVGH" class="2">
+<segment>
+<wire x1="-76.2" y1="25.4" x2="-71.12" y2="25.4" width="0.1524" layer="91"/>
+<label x="-71.12" y="25.4" size="1.016" layer="95" xref="yes"/>
+<pinref part="D5" gate="G$1" pin="K"/>
+</segment>
 <segment>
 <wire x1="-162.56" y1="-7.62" x2="-154.94" y2="-7.62" width="0.1524" layer="91"/>
@@
 </segment>
 </net>
-<net name="PREVGH" class="2">
-<segment>
-<wire x1="-76.2" y1="25.4" x2="-71.12" y2="25.4" width="0.1524" layer="91"/>
-<label x="-71.12" y="25.4" size="1.016" layer="95" xref="yes"/>
-<pinref part="D5" gate="G$1" pin="K"/>
-</segment>
-</net>
