File: Hardware/Proiect_TSC_2025 v63.brd (EAGLE design)
At the start: 170 x 111.2 mm, 103 parts, among them IC1 BD5229G-TR, IC4 XC6220A331MR-G, J1 FH34SRJ-24S-0.5SH_99_, J2 SAMACSYS_PARTS_USB4110-GF-A, J3 QWIIC_RIGHT_ANGLE, J4 112A-TAAR-R03_ATTEND, Q1 20V/4.2A/52mΩ/1.4W, Q2 20V/4.2A/52mΩ/1.4W, Q3 SI1308EDL-T1-GE3, U1 W25Q512JVEIQ, U2 ESP32-C6-WROOM-1-N8, U3 DS3231SN#, U4 MAX17048G+T10

Commit message: Fixed issues
Parts:
- moved J3 4.20 mm to (165.6, 18.1), turned to 270 degrees
- moved U2 1.80 mm to (12.8, 45.2)
Connections:
- removed net N$4: EPD_C9.2, J1.21
- net PREVGH: now also EPD_C9.2, J1.21
Routing:
- net PREVGH: track 0.00 -> 22.9 mm, vias 0 -> 2
- net GND: track 682.7 -> 702.3 mm
- net GDR: track 65.1 -> 49.6 mm, vias 0 -> 3
- net N$4: track 14.2 -> 0.00 mm, vias 2 -> 0
- net SCL: track 206.9 -> 194.3 mm, vias 8 -> 7
- net USB_D+: track 137.1 -> 149.5 mm
- net EPD_DC: track 166.7 -> 177.7 mm
- net EPD_RST: track 167.9 -> 178.2 mm, vias 5 -> 4
- net FLASH_CS: track 59.5 -> 66.0 mm
- net EPD_CS: track 194.6 -> 189.3 mm, vias 8 -> 7
- net N$2: track 69.7 -> 66.0 mm, vias 2 -> 5
- net USB_D-: track 146.5 -> 149.8 mm
- net N$9: track 17.1 -> 14.4 mm, vias 0 -> 2
- net 32KHZ: track 74.9 -> 77.7 mm
- net MOSI: track 152.3 -> 155.0 mm
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- added copper zone on layer 16, net BOTTOM
- removed copper zone on layer 16, net TOP
Other:
- outline, holes or cut-outs redrawn
